File: vca/debug.kicad_sch (KiCad schematic)
At the start: 1 part

Commit message: working on front panel
Parts:
- J2: value (none) -> Conn_ARM_JTAG_SWD_10; footprint (none) -> Connector_PinHeader_2.54mm:PinHeader_2x05_P2.54mm_Vertical
Changed lines of the file:
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@@
       (effects (font (size 1.27 1.27)) (justify right))
     )
-    (property "Value" "" (id 1) (at 46.99 45.0849 0)
+    (property "Value" "Conn_ARM_JTAG_SWD_10" (id 1) (at 46.99 45.0849 0)
       (effects (font (size 1.27 1.27)) (justify right))
     )
-    (property "Footprint" "" (id 2) (at 59.055 43.815 0)
+    (property "Footprint" "Connector_PinHeader_2.54mm:PinHeader_2x05_P2.54mm_Vertical" (id 2) (at 59.055 43.815 0)
       (effects (font (size 1.27 1.27)) hide)
     )
@@
       (effects (font (size 1.27 1.27)) hide)
     )
-    (property "Value" "" (id 1) (at 59.055 66.04 0))
+    (property "Value" "GND" (id 1) (at 59.055 66.04 0))
     (property "Footprint" "" (id 2) (at 59.055 60.96 0)
       (effects (font (size 1.27 1.27)) hide)
@@
       (effects (font (size 1.27 1.27)) hide)
     )
-    (property "Value" "" (id 1) (at 59.055 20.32 0))
+    (property "Value" "+3V3" (id 1) (at 59.055 20.32 0))
     (property "Footprint" "" (id 2) (at 59.055 26.035 0)
       (effects (font (size 1.27 1.27)) hide)
