File: vca/vca.kicad_pcb (KiCad board)
At the start: 2 copper layers, 2 x 2 mm, 120 parts, among them J2 Conn_ARM_JTAG_SWD_10, U1 LM324, U10 LUM-1502-03_3.5mm_mono_vertic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, U11 LUM-1502-03_3.5mm_mono_vertic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, U12 LUM-1502-03_3.5mm_mono_vertic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, U13 LUM-1502-03_3.5mm_mono_vertic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, U14 LUM-1502-03_3.5mm_mono_vertic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, U15 LUM-1502-03_3.5mm_mono_vertic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, U16 power_conn_16, U17 LUM-1502-03_3.5mm_mono_vertic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, U18 LM7805_TO220, U19 ZLDO1117G33TA, U2 LM324, U20 LUM-1502-03_3.5mm_mono_vertic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, U3 LM324, U4 STM32F103C6Tx, U5 TL074, U6 TL074, U7 TLC7528, U8 LUM-1502-03_3.5mm_mono_vertic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, U9 LUM-1502-03_3.5mm_mono_vertic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, Y1 Crystal_8Mhz

Commit message: working on the PCB
Parts:
- added CON_BACK1: 2_15_Back_Front_Conn_70, eurorack:2_15_back_front_conn_70, F.Cu at (55.0, 15.0)
- added CON_FRONT1: 2_15_Back_Front_Conn_70, eurorack:2_15_back_front_conn_70, F.Cu at (5.00, 15.0)
- added R42: R-1k-1206, Resistor_SMD:R_1206_3216Metric_Pad1.30x1.75mm_HandSolder, B.Cu at (34.8, 19.8)
- added R43: R-1k-1206, Resistor_SMD:R_1206_3216Metric_Pad1.30x1.75mm_HandSolder, B.Cu at (34.8, 36.9)
- added R44: R-1k-1206, Resistor_SMD:R_1206_3216Metric_Pad1.30x1.75mm_HandSolder, B.Cu at (34.9, 54.2)
- added R45: R-1k-1206, Resistor_SMD:R_1206_3216Metric_Pad1.30x1.75mm_HandSolder, B.Cu at (34.9, 71.4)
- added R46: R-1k-1206, Resistor_SMD:R_1206_3216Metric_Pad1.30x1.75mm_HandSolder, B.Cu at (34.8, 2.69)
- added R47: R-1k-1206, Resistor_SMD:R_1206_3216Metric_Pad1.30x1.75mm_HandSolder, B.Cu at (37.2, 19.8)
- added R48: R-1k-1206, Resistor_SMD:R_1206_3216Metric_Pad1.30x1.75mm_HandSolder, B.Cu at (37.2, 36.9)
- added R49: R-1k-1206, Resistor_SMD:R_1206_3216Metric_Pad1.30x1.75mm_HandSolder, B.Cu at (37.2, 54.2)
- added R50: R-1k-1206, Resistor_SMD:R_1206_3216Metric_Pad1.30x1.75mm_HandSolder, B.Cu at (37.2, 71.4)
- added R51: R-1k-1206, Resistor_SMD:R_1206_3216Metric_Pad1.30x1.75mm_HandSolder, B.Cu at (37.2, 2.69)
- D10, D4, D5, D9, R16, R17, R18, R19, R20, R21, R31, R32, R33, R34, R35, R36, U1, U2, U3: moved to B.Cu
- U10, U11, U12, U13, U14, U15, U17, U20, U8, U9: footprint eurorack:LUM 1502-03 -> eurorack:LUM 1502-03 LED
- moved RV7 180.3 mm to (20.7, 46.1), turned to 90 degrees
- moved U14 177.9 mm to (40.8, 41.4)
- moved RV5 171.6 mm to (8.24, 11.7), turned to 90 degrees
- moved RV6 168.4 mm to (20.7, 28.9), turned to 90 degrees
- moved U12 168.1 mm to (30.1, 7.17)
- moved U13 166.9 mm to (40.8, 24.2)
- moved RV1 156.1 mm to (8.24, 28.9), turned to 90 degrees
- moved U8 154.1 mm to (30.1, 24.2)
- moved RV2 147.8 mm to (8.24, 46.1), turned to 90 degrees
- moved U9 144.4 mm to (30.1, 41.4)
- moved U20 138.9 mm to (40.8, 7.11)
- moved RV10 138.6 mm to (20.7, 11.7), turned to 90 degrees
- moved RV3 135.3 mm to (8.24, 63.3), turned to 90 degrees
- moved U10 131.0 mm to (30.1, 58.6)
- moved R18 120.5 mm to (32.1, 48.1), turned to 180 degrees
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Connections:
- C12 pad 1: +5V -> +5C
- C12 pad 2: GND -> GND2
- C13 pad 1: +5V -> +5C
- C13 pad 2: GND -> GND2
- C14 pad 1: +5V -> +5C
- C14 pad 2: GND -> GND2
- IN_A1 pad T: /DAC/InA -> F_INA
- IN_B1 pad T: /DAC/InB -> F_INB
- IN_B1 pad TN: unconnected-(IN_B1-PadTN) -> +10V
- J2 pad 2: AIN_A1_LED -> B_AIN_A1_LED
- J2 pad 4: AIN_D1_LED -> B_AIN_D1_LED
- J2 pad 8: AIN_S1_LED -> B_AIN_S1_LED
- OUT_A1 pad T: /DAC/OutA -> F_OUTA
- OUT_A1 pad TN: /DAC/OutA -> F_OUTA
- OUT_B1 pad T: /DAC/OutB -> F_OUTB
- OUT_B1 pad TN: /DAC/OutB -> F_OUTB
- R11 pad 2: GND -> GND2
- R12 pad 1: +12VA -> +12C
- R14 pad 2: GND -> GND2
- R15 pad 1: +12VA -> +12C
- R16 pad 1: +12VA -> +12C
- R18 pad 2: GND -> GND2
- R19 pad 1: +12VA -> +12C
- R21 pad 2: GND -> GND2
- R22 pad 1: +12VA -> +12C
- R24 pad 2: GND -> GND2
- R25 pad 1: +12VA -> +12C
- R27 pad 2: GND -> GND2
- R28 pad 1: +12VA -> +12C
- R30 pad 2: GND -> GND2
- R31 pad 1: +12VA -> +12C
- R33 pad 2: GND -> GND2
- R34 pad 1: +12VA -> +12C
- R36 pad 2: GND -> GND2
- R37 pad 1: +12VA -> +12C
- R39 pad 2: GND -> GND2
- RV1 pad 11: GND -> GND2
- RV1 pad 2: AIN_A0 -> F_AIN_A0
- RV1 pad 3: GND -> GND2
- RV1 pad 4: AIN_A0_LED -> F_AIN_A0_LED
- RV1 pad 7: GND -> GND2
- RV1 pad 8: AIN_A0_LED -> F_AIN_A0_LED
- RV10 pad 11: GND -> GND2
- RV10 pad 2: AIN_T1 -> F_AIN_T1
- RV10 pad 3: GND -> GND2
- RV10 pad 4: AIN_T1_LED -> F_AIN_T1_LED
- RV10 pad 7: GND -> GND2
- RV10 pad 8: AIN_T1_LED -> F_AIN_T1_LED
- RV2 pad 11: GND -> GND2
- RV2 pad 2: AIN_D0 -> F_AIN_D0
- RV2 pad 3: GND -> GND2
- RV2 pad 4: AIN_D0_LED -> F_AIN_D0_LED
- RV2 pad 7: GND -> GND2
- RV2 pad 8: AIN_D0_LED -> F_AIN_D0_LED
- RV3 pad 11: GND -> GND2
- RV3 pad 2: AIN_S0 -> F_AIN_S0
- RV3 pad 3: GND -> GND2
- RV3 pad 4: AIN_S0_LED -> F_AIN_S0_LED
- RV3 pad 7: GND -> GND2
- RV3 pad 8: AIN_S0_LED -> F_AIN_S0_LED
- RV4 pad 11: GND -> GND2
- RV4 pad 2: AIN_R0 -> F_AIN_R0
- RV4 pad 3: GND -> GND2
- RV4 pad 4: AIN_R0_LED -> F_AIN_R0_LED
- RV4 pad 7: GND -> GND2
- RV4 pad 8: AIN_R0_LED -> F_AIN_R0_LED
- RV5 pad 11: GND -> GND2
- RV5 pad 2: AIN_T0 -> F_AIN_T0
- RV5 pad 3: GND -> GND2
- RV5 pad 4: AIN_T0_LED -> F_AIN_T0_LED
- RV5 pad 7: GND -> GND2
- RV5 pad 8: AIN_T0_LED -> F_AIN_T0_LED
- RV6 pad 11: GND -> GND2
- RV6 pad 2: AIN_A1 -> F_AIN_A1
- RV6 pad 3: GND -> GND2
- RV6 pad 4: AIN_A1_LED -> F_AIN_A1_LED
- RV6 pad 7: GND -> GND2
- RV6 pad 8: AIN_A1_LED -> F_AIN_A1_LED
- RV7 pad 11: GND -> GND2
- RV7 pad 2: AIN_D1 -> F_AIN_D1
- RV7 pad 3: GND -> GND2
- RV7 pad 4: AIN_D1_LED -> F_AIN_D1_LED
- RV7 pad 7: GND -> GND2
- RV7 pad 8: AIN_D1_LED -> F_AIN_D1_LED
- RV8 pad 11: GND -> GND2
- RV8 pad 2: AIN_S1 -> F_AIN_S1
- RV8 pad 3: GND -> GND2
- RV8 pad 4: AIN_S1_LED -> F_AIN_S1_LED
- RV8 pad 7: GND -> GND2
- RV8 pad 8: AIN_S1_LED -> F_AIN_S1_LED
- RV9 pad 11: GND -> GND2
- RV9 pad 2: AIN_R1 -> F_AIN_R1
- RV9 pad 3: GND -> GND2
- RV9 pad 4: AIN_R1_LED -> F_AIN_R1_LED
- RV9 pad 7: GND -> GND2
- RV9 pad 8: AIN_R1_LED -> F_AIN_R1_LED
- U1 pad 11: GND -> GND2
- U1 pad 4: +5V -> +5C
- U10 pad S: GND -> GND2
- U11 pad S: GND -> GND2
- U12 pad S: GND -> GND2
- U13 pad S: GND -> GND2
- U14 pad S: GND -> GND2
- U15 pad S: GND -> GND2
- U17 pad S: GND -> GND2
- U2 pad 11: GND -> GND2
- U2 pad 4: +5V -> +5C
- U20 pad S: GND -> GND2
- U3 pad 10: GND -> GND2
- U3 pad 11: GND -> GND2
- U3 pad 12: GND -> GND2
- U3 pad 4: +5V -> +5C
- U4 pad 10: AIN_A0 -> B_AIN_A0
- U4 pad 11: AIN_D0 -> B_AIN_D0
- U4 pad 12: AIN_S0 -> B_AIN_S0
- U4 pad 13: AIN_R0 -> B_AIN_R0
- U4 pad 14: AIN_A1 -> B_AIN_A1
- U4 pad 15: AIN_D1 -> B_AIN_D1
- U4 pad 16: AIN_S1 -> B_AIN_S1
- U4 pad 17: AIN_R1 -> B_AIN_R1
- U4 pad 18: AIN_T0 -> B_AIN_T0
- U4 pad 19: AIN_T1 -> B_AIN_T1
- U4 pad 27: AIN_T1_LED -> B_AIN_T1_LED
- U4 pad 28: AIN_R1_LED -> B_AIN_R1_LED
- U4 pad 29: AIN_A0_LED -> B_AIN_A0_LED
- U4 pad 30: AIN_D0_LED -> B_AIN_D0_LED
- U4 pad 31: AIN_S0_LED -> B_AIN_S0_LED
- U4 pad 32: AIN_R0_LED -> B_AIN_R0_LED
- U4 pad 33: AIN_T0_LED -> B_AIN_T0_LED
- U4 pad 34: AIN_A1_LED -> B_AIN_A1_LED
- U4 pad 37: AIN_D1_LED -> B_AIN_D1_LED
- U4 pad 38: AIN_S1_LED -> B_AIN_S1_LED
- U5 pad 1: /DAC/OutA -> B_OUTA
- U5 pad 10: /DAC/InA -> B_INA
- U5 pad 2: /DAC/OutA -> B_OUTA
- U6 pad 1: /DAC/OutB -> B_OUTB
- U6 pad 10: /DAC/InB -> B_INB
- U6 pad 2: /DAC/OutB -> B_OUTB
- U8 pad S: GND -> GND2
- U9 pad S: GND -> GND2
Routing:
- net GND: track 0.00 -> 2.66 mm, vias 0 -> 1
- added copper zone on B.Cu, net GND
- added copper zone on F.Cu, net GND
- added copper zone on In1.Cu, net GND
- added copper zone on In2.Cu, net GND
- added copper zone on B.Cu, net GND2
- added copper zone on F.Cu, net GND2
- added copper zone on In1.Cu, net GND2
- added copper zone on In2.Cu, net GND2
Other:
- board size 2 x 2 mm -> 95 x 100 mm
- copper layers 2 -> 4
- board text added: "10 HP, 50.50mm"
- board text added: "x+50"

Commit message: working on front panel
Parts:
- D1, D3, D6, D7, D8, R10, R11, R12, R13, R14, R15, R22, R23, R24, R25, R26, R27, R28, R29, R3, R30, R4, R5, R6: moved to B.Cu
- moved R24 218.4 mm to (20.8, 3.28), turned to 45 degrees
- moved R27 213.9 mm to (34.7, 8.46), turned to 90 degrees
- moved R23 207.1 mm to (26.1, 3.86)
- moved D6 207.0 mm to (26.2, 1.55), turned to 180 degrees
- moved R26 205.2 mm to (37.1, 12.1), turned to 180 degrees
- moved R22 204.7 mm to (27.1, 11.9)
- moved R25 203.7 mm to (35.2, 29.1), turned to 90 degrees
- moved R30 201.8 mm to (37.7, 30.6), turned to 90 degrees
- moved D7 197.5 mm to (43.8, 15.6), turned to 90 degrees
- moved R28 197.0 mm to (36.3, 46.0)
- moved D8 192.6 mm to (41.1, 34.3)
- moved R29 191.7 mm to (41.4, 32.0), turned to 180 degrees
- moved R11 190.2 mm to (22.3, 19.1), turned to -90 degrees
- moved R12 183.0 mm to (26.5, 38.7), turned to -90 degrees
- moved R14 182.6 mm to (34.1, 32.1)
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Connections:
- CON_BACK1 pad 16: unconnected-(CON_BACK1-Pad16) -> B_+10V
- CON_BACK1 pad 17: unconnected-(CON_BACK1-Pad17) -> B_INA
- CON_BACK1 pad 18: unconnected-(CON_BACK1-Pad18) -> +12V
- CON_BACK1 pad 19: unconnected-(CON_BACK1-Pad19) -> B_OUTA
- CON_BACK1 pad 20: unconnected-(CON_BACK1-Pad20) -> B_AIN_R0_LED
- CON_BACK1 pad 21: unconnected-(CON_BACK1-Pad21) -> B_AIN_R0
- CON_BACK1 pad 26: unconnected-(CON_BACK1-Pad26) -> B_INB
- CON_BACK1 pad 30: unconnected-(CON_BACK1-Pad30) -> B_OUTB
- CON_FRONT1 pad 16: unconnected-(CON_FRONT1-Pad16) -> +10V
- CON_FRONT1 pad 17: unconnected-(CON_FRONT1-Pad17) -> F_INA
- CON_FRONT1 pad 18: unconnected-(CON_FRONT1-Pad18) -> +12VA
- CON_FRONT1 pad 19: unconnected-(CON_FRONT1-Pad19) -> F_OUTA
- CON_FRONT1 pad 20: unconnected-(CON_FRONT1-Pad20) -> F_AIN_R0_LED
- CON_FRONT1 pad 21: unconnected-(CON_FRONT1-Pad21) -> F_AIN_R0
- CON_FRONT1 pad 26: unconnected-(CON_FRONT1-Pad26) -> F_INB
- CON_FRONT1 pad 30: unconnected-(CON_FRONT1-Pad30) -> F_OUTB
- OUT_A1 pad LA: GND -> Net-(OUT_A1-PadLA)
- OUT_A1 pad LK: Net-(OUT_A1-PadLK) -> GND
- OUT_B1 pad LA: GND -> Net-(OUT_B1-PadLA)
- OUT_B1 pad LK: Net-(OUT_B1-PadLK) -> GND
- R5 pad 1: Net-(OUT_A1-PadLK) -> Net-(OUT_A1-PadLA)
- R6 pad 1: Net-(OUT_B1-PadLK) -> Net-(OUT_B1-PadLA)
- U6 pad 6: +10V -> B_+10V
- U6 pad 7: +10V -> B_+10V
Routing:
- net +10V: track 0.00 -> 42.9 mm
- net F_AIN_R0: track 0.00 -> 25.3 mm
- net F_OUTA: track 0.00 -> 20.8 mm
- net Net-(RV4-Pad1): track 0.00 -> 20.1 mm, vias 0 -> 1
- net F_AIN_R0_LED: track 0.00 -> 18.9 mm
- net +12VA: track 0.00 -> 16.2 mm, vias 0 -> 2
- net F_OUTB: track 0.00 -> 15.3 mm
- net Net-(OUT_B1-PadLA): track 0.00 -> 7.47 mm
- net F_INA: track 0.00 -> 5.54 mm
- net F_INB: track 0.00 -> 5.26 mm
- net Net-(RV3-Pad1): track 0.00 -> 4.36 mm
- net Net-(IN_A1-PadLA): track 0.00 -> 3.90 mm
- net Net-(OUT_A1-PadLA): track 0.00 -> 3.79 mm
- net Net-(IN_B1-PadLA): track 0.00 -> 3.57 mm
- net Net-(RV4-Pad5): track 0.00 -> 3.11 mm, vias 0 -> 1
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
Commit message: working on the front panel
Connections:
- CON_BACK1 pad 16: B_+10V -> B_AIN_S0
- CON_BACK1 pad 17: B_INA -> B_+10V
- CON_BACK1 pad 18: +12V -> B_INA
- CON_BACK1 pad 19: B_OUTA -> +12V
- CON_BACK1 pad 20: B_AIN_R0_LED -> B_OUTA
- CON_BACK1 pad 21: B_AIN_R0 -> B_AIN_R0_LED
- CON_BACK1 pad 22: unconnected-(CON_BACK1-Pad22) -> B_AIN_S0_LED
- CON_BACK1 pad 23: unconnected-(CON_BACK1-Pad23) -> B_AIN_R0
- CON_BACK1 pad 24: unconnected-(CON_BACK1-Pad24) -> B_AIN_R1
- CON_BACK1 pad 25: unconnected-(CON_BACK1-Pad25) -> B_AIN_R1_LED
- CON_BACK1 pad 26: B_INB -> B_AIN_S1
- CON_BACK1 pad 27: unconnected-(CON_BACK1-Pad27) -> B_AIN_S1_LED
- CON_BACK1 pad 28: unconnected-(CON_BACK1-Pad28) -> B_INB
- CON_BACK1 pad 29: unconnected-(CON_BACK1-Pad29) -> B_AIN_D1_LED
- CON_FRONT1 pad 16: +10V -> F_AIN_S0
- CON_FRONT1 pad 17: F_INA -> +10V
- CON_FRONT1 pad 18: +12VA -> F_INA
- CON_FRONT1 pad 19: F_OUTA -> +12VA
- CON_FRONT1 pad 20: F_AIN_R0_LED -> F_OUTA
- CON_FRONT1 pad 21: F_AIN_R0 -> F_AIN_R0_LED
- CON_FRONT1 pad 22: unconnected-(CON_FRONT1-Pad22) -> F_AIN_S0_LED
- CON_FRONT1 pad 23: unconnected-(CON_FRONT1-Pad23) -> F_AIN_R0
- CON_FRONT1 pad 24: unconnected-(CON_FRONT1-Pad24) -> F_AIN_R1
- CON_FRONT1 pad 25: unconnected-(CON_FRONT1-Pad25) -> F_AIN_R1_LED
- CON_FRONT1 pad 26: F_INB -> F_AIN_S1
- CON_FRONT1 pad 27: unconnected-(CON_FRONT1-Pad27) -> F_AIN_S1_LED
- CON_FRONT1 pad 28: unconnected-(CON_FRONT1-Pad28) -> F_INB
- CON_FRONT1 pad 29: unconnected-(CON_FRONT1-Pad29) -> F_AIN_D1_LED
Routing:
- net F_AIN_D1_LED: track 0.00 -> 76.1 mm, vias 0 -> 2
- net Net-(R17-Pad2): track 0.00 -> 49.2 mm
- net F_AIN_S0_LED: track 0.00 -> 47.0 mm
- net F_AIN_S1: track 0.00 -> 41.8 mm
- net F_AIN_S1_LED: track 0.00 -> 41.3 mm
- net Net-(R35-Pad2): track 0.00 -> 33.8 mm, vias 0 -> 2
- net F_AIN_S0: track 0.00 -> 33.3 mm
- net GND2: track 0.00 -> 22.7 mm, vias 0 -> 7
- net Net-(RV8-Pad1): track 0.00 -> 20.9 mm, vias 0 -> 1
- net F_AIN_R1_LED: track 0.00 -> 19.6 mm
- net F_AIN_R1: track 0.00 -> 19.5 mm
- net Net-(RV7-Pad1): track 0.00 -> 9.07 mm, vias 0 -> 1
- net Net-(R50-Pad2): track 0.00 -> 7.96 mm
- net Net-(R45-Pad2): track 0.00 -> 7.70 mm
- net Net-(R44-Pad2): track 0.00 -> 7.64 mm
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
Commit message: working on the front
Parts:
- R37, R38, R39: moved to B.Cu
- moved R37 162.5 mm to (23.9, 11.2), turned to 90 degrees
- moved R39 155.5 mm to (32.5, 17.3), turned to 180 degrees
- moved R38 144.7 mm to (39.9, 17.3), turned to 180 degrees
- moved D11 141.1 mm to (43.5, 15.3), turned to -90 degrees
- moved R42 4.52 mm to (34.7, 24.3)
- moved R47 1.14 mm to (36.6, 20.7), turned to -45 degrees
Connections:
- CON_BACK1 pad 1: unconnected-(CON_BACK1-Pad1) -> B_AIN_T0
- CON_BACK1 pad 2: unconnected-(CON_BACK1-Pad2) -> B_AIN_A0
- CON_BACK1 pad 3: unconnected-(CON_BACK1-Pad3) -> B_AIN_T0_LED
- CON_BACK1 pad 4: unconnected-(CON_BACK1-Pad4) -> B_AIN_T1_LED
- CON_BACK1 pad 5: unconnected-(CON_BACK1-Pad5) -> B_AIN_D0
- CON_BACK1 pad 6: unconnected-(CON_BACK1-Pad6) -> B_AIN_A0_LED
- CON_BACK1 pad 7: unconnected-(CON_BACK1-Pad7) -> B_AIN_D0_LED
- CON_BACK1 pad 8: unconnected-(CON_BACK1-Pad8) -> B_AIN_A1
- CON_FRONT1 pad 1: unconnected-(CON_FRONT1-Pad1) -> F_AIN_T0
- CON_FRONT1 pad 2: unconnected-(CON_FRONT1-Pad2) -> F_AIN_A0
- CON_FRONT1 pad 3: unconnected-(CON_FRONT1-Pad3) -> F_AIN_T0_LED
- CON_FRONT1 pad 4: unconnected-(CON_FRONT1-Pad4) -> F_AIN_T1_LED
- CON_FRONT1 pad 5: unconnected-(CON_FRONT1-Pad5) -> F_AIN_D0
- CON_FRONT1 pad 6: unconnected-(CON_FRONT1-Pad6) -> F_AIN_A0_LED
- CON_FRONT1 pad 7: unconnected-(CON_FRONT1-Pad7) -> F_AIN_D0_LED
- CON_FRONT1 pad 8: unconnected-(CON_FRONT1-Pad8) -> F_AIN_A1
Routing:
- net F_AIN_D0_LED: track 0.00 -> 44.2 mm, vias 0 -> 1
- net Net-(R23-Pad2): track 0.00 -> 42.0 mm
- net F_AIN_D0: track 0.00 -> 26.0 mm
- net Net-(RV10-Pad1): track 0.00 -> 25.0 mm, vias 0 -> 1
- net F_AIN_A0_LED: track 0.00 -> 23.3 mm
- net Net-(R37-Pad2): track 0.00 -> 17.8 mm, vias 0 -> 1
- net Net-(D11-Pad1): track 0.00 -> 17.0 mm
- net F_AIN_T0_LED: track 0.00 -> 15.6 mm
- net GND2: track 22.7 -> 37.8 mm, vias 7 -> 10
- net F_AIN_T0: track 0.00 -> 13.6 mm
- net F_AIN_A1_LED: track 0.00 -> 8.52 mm
- net Net-(R51-Pad2): track 0.00 -> 7.76 mm
- net F_AIN_T1_LED: track 0.00 -> 7.39 mm
- net Net-(R46-Pad2): track 0.00 -> 7.24 mm
- net Net-(R47-Pad2): track 0.00 -> 7.10 mm
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
Commit message: working on the back panel power section
Parts:
- C10: value C-2u2-1812 -> C-100nF-0805; footprint Capacitor_SMD:C_1812_4532Metric_Pad1.57x3.40mm_HandSolder -> Capacitor_SMD:C_0805_2012Metric_Pad1.18x1.45mm_HandSolder; moved to B.Cu
- C21, C22, C29, C30, C4, C5, C6, C7, J2, U16, U18: moved to B.Cu
- moved C12 115.2 mm to (14.5, 33.2)
- moved J2 107.5 mm to (77.0, 28.3), turned to -135 degrees
- moved C14 95.8 mm to (13.0, 66.4), turned to 180 degrees
- moved C13 95.4 mm to (23.7, 49.7), turned to 90 degrees
- moved C22 87.7 mm to (53.6, 70.8), turned to 90 degrees
- moved C30 80.3 mm to (54.7, 75.9)
- moved U19 74.3 mm to (57.9, 70.9)
- moved C4 70.2 mm to (69.2, 42.2)
- moved C31 69.7 mm to (55.8, 76.1)
- moved C5 69.1 mm to (75.1, 36.9)
- moved JP2 68.4 mm to (53.4, 81.0), turned to 180 degrees
- moved U18 62.0 mm to (62.6, 81.1), turned to 180 degrees
- moved C21 61.1 mm to (67.6, 75.6), turned to 90 degrees
- moved R2 57.6 mm to (63.5, 56.0), turned to 135 degrees
- moved U4 57.3 mm to (73.9, 44.4), turned to 45 degrees
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Connections:
- C21 pad 1: +5V -> Net-(C21-Pad1)
- CON_BACK1 pad 10: unconnected-(CON_BACK1-Pad10) -> B_AIN_T1
- CON_BACK1 pad 9: unconnected-(CON_BACK1-Pad9) -> B_AIN_A1_LED
- CON_FRONT1 pad 10: unconnected-(CON_FRONT1-Pad10) -> F_AIN_T1
- CON_FRONT1 pad 9: unconnected-(CON_FRONT1-Pad9) -> F_AIN_A1_LED
- JP2 pad 1: Net-(JP2-Pad1) -> Net-(C21-Pad1)
- U18 pad 3: Net-(JP2-Pad1) -> Net-(C21-Pad1)
Routing:
- net +5V: track 0.00 -> 56.7 mm
- net +12V: track 0.00 -> 39.2 mm
- net GND: track 8.54 -> 44.6 mm, vias 6 -> 13
- net -12V: track 0.00 -> 24.5 mm
- net GND2: track 37.8 -> 61.9 mm, vias 10 -> 12
- net +3V3: track 0.00 -> 23.0 mm, vias 0 -> 35
- net F_AIN_T1: track 0.00 -> 19.1 mm
- net +5C: track 0.00 -> 16.1 mm, vias 0 -> 3
- net Net-(C21-Pad1): track 0.00 -> 16.0 mm
- net Net-(C1-Pad1): track 0.00 -> 15.5 mm
- net F_AIN_A1_LED: track 8.52 -> 20.8 mm, vias 0 -> 1
- net Net-(R2-Pad2): track 0.00 -> 11.5 mm
- net F_AIN_T1_LED: track 7.39 -> 15.9 mm
- net Net-(C2-Pad1): track 0.00 -> 5.91 mm
- net Net-(R23-Pad2): track 42.0 -> 44.9 mm
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- added copper zone on B.Cu, net +3V3
- added copper zone on F.Cu, net +3V3
- added copper zone on In1.Cu, net +3V3
- added copper zone on In2.Cu, net +3V3
